Commit message: 存檔：滾輪物理撿球成功版本，取代「碰到就刪除球」，run76/77 皆 9/9 進後車廂
- 原因：影片 47.webm 成功時滾輪在 record 筆記的位置 (y=0.2, z=0.03)，後來被改回
  CAD 位置 (0.102, 0.045)，離後車廂 17.7cm 前擋牆只剩 10cm，球被推到牆邊只能垂直
  彈起 (experiments/roller_pickup 實測)。URDF 滾輪改回 (0.2, 0.03)，恢復滾輪碰撞
  (半徑 0.045)，滾輪關節加進 joint_states。
- 掃描 W(/roller_cmd angular.z)=35~55 × 盲衝 0.2~0.4 m/s：W=40/45 全部進車廂，
  W>=50 拋過頭飛出車尾，W=35 邊緣；採用 W=42.5 (約 66 rad/s) 常轉。
- grid_patrol_node：移除 DeleteEntity，「撿到」改用 Gazebo 真實座標判定球躺在
  後車廂地板 (x∈[-0.36,0]、y 在車廂寬度內、z 0.05~0.15) 連續 3 次；結束時稽核
  每顆球的最終位置。
- 里程計影響：run77 位置誤差平均 0.078m/最大 0.184m，航向 0.63°，比無碰撞的
  run74 (0.026m/0.17°) 略大，誤差在前 60 秒追球期間累積後持平。

Co-Authored-By: Claude Fable 5.1 <noreply@anthropic.com>

File: experiments/roller_pickup/simple_bot_roller_collision.urdf (robot description, URDF)
Before this commit: robot tennis_bot, 11 links, 10 joints
Joints:
- joint left_roller_joint: origin xyz=0.065 0.2 0.03 rpy=-0.785398 0 0 -> xyz=0.065 0.102322 0.045104 rpy=-0.785398 0 0
- joint right_roller_joint: origin xyz=0.205 0.2 0.03 rpy=-0.785398 0 0 -> xyz=0.205 0.102322 0.045104 rpy=-0.785398 0 0
