Commit message: 8/16 問題出在延遲通訊
存檔點：陀螺儀+輪速里程計、左右滾輪判定、目標鎖定 (SAME_BALL_PX=150，即時放開
不等待)、MIN_CONTOUR_AREA=55px²、原路倒車機制(關閉)、debug用的target_ball_guess
估測、run1~run24實驗數據。

目前定位到的問題：_joint_state_cb 用真實時鐘(wall clock)算 dt，當模擬即時率
掉下去 (懷疑是 Gazebo GUI 渲染 + 密集非同步服務查詢同時搶資源造成)，dt 可能
超過 0.5 秒防呆門檻，導致該次陀螺儀積分被整段跳過，車體真實有轉動/移動但
里程計沒記錄到，這是目前找到的位置誤差主要來源之一。下一步：加 debug log
確認真的是即時率問題，如果是，改用模擬時間 (/clock) 算 dt 才是根本解法。

Co-Authored-By: Claude Sonnet 5 <noreply@anthropic.com>

File: src/tennis_bot/urdf/simple_bot.urdf (robot description, URDF)
Before this commit: robot tennis_bot, 10 links, 9 joints
Links:
- added link imu_link, mass 0.001
- link left_roller: geometry visual box size=0.01 0.01 0.01; visual cylinder length=0.04 radius=0.05
- link right_roller: geometry visual box size=0.01 0.01 0.01; visual cylinder length=0.04 radius=0.05
Joints:
- added joint imu_joint: type fixed, parent base_link, child imu_link, origin xyz=0 -0.135 0 rpy=0 0 0

Commit message: 相機對應 D 同學實測校正 + 視覺輸出節奏照實體 CSV 精確化
- 焦距/視角：D 程式 FOCAL 390 (512 寬) -> 水平視角 80° 改 66.6°；球輪廓門檻 55/15 -> 90/25 維持 3 m
- 光軸偏移：D 程式 image_cx=283 -> 相機往左偏 3.96°，vision 用第 353.75 行當正前方 (邊界左右也以此分)
- D 同學 6/21 靜態測試：距離 ×0.944 + 1% 雜訊、角度 0.6° 雜訊
- 視覺輸出節奏 (5 個 run、3199 連續幀)：短 0.1107±0.0037 s、長 0.4525±0.0308 s 嚴格「短短長」
- 弓字格邊長隨相機視角 3.09 -> 2.63 m (每半場 25 格)
- 孿生準確度表 v2：Kp0.6 上升 2.03 s/overshoot 5.1° (實體 2.0~3.3 s/1.4~7.9°)、Kp1.5 擺幅 21.8° (實體 18~30°)
  都落在實體範圍內；Kp0.3 4.74 s 仍略快 (實體 5.3~7.6 s)
- 回歸：全場 run161 9/9 448.9 s (+15%)、半場 135° run162 10/10 398.0 s (+45%，視角變窄看到的球變少)
- 延遲補償 Kp0.6 (舊相機)：穩定 2.94 s、0° (無補償 5.74 s、4.3°)

Co-Authored-By: Claude Opus 5.5 <noreply@anthropic.com>

File: src/tennis_bot/urdf/simple_bot.urdf (robot description, URDF)
Before this commit: robot tennis_bot, 11 links, 10 joints
Joints:
- joint camera_joint: origin xyz=0.135 0.1 0.13 rpy=0 0 1.5708 -> xyz=0.135 0.1 0.13 rpy=0 0 1.6399

Commit message: 實體車模式：模擬直接跑 D 同學 Jetson 程式 + B 同學 main.c，鏡頭/場地照實測校正
- jetson_d/：D 同學 10/11 版程式原檔 (md5 同 Jetson) + YOLO ONNX；jetson_d_code.py 用 ast 取出不碰硬體的函式
- jetson_d_node：D 主迴圈 SIL (黃線 yellow_runtime、YOLO onnxruntime、EdgeUartGate)，迴圈時間照 10/11 CSV 抽樣，
  V4L2 4 buffer 相機緩衝區模型 (推算畫面延遲中位數約 0.42~0.47 s，未實測)
- stm32_b_node：B 同學 10/12「加入邊界判斷版本」main.c 移植 (避線 > 追球 > 巡邏，TurnPrecise ±240/-360，點放追球)，
  可切換 Sean 的 P 轉向；real_car_node 只當裁判 (起點、撿球判定、軌跡)
- URDF 鏡頭：10/02 實測擬合離地 20.2 cm、俯角 21.3° (原本 15 cm 水平)；x 放滾輪軸上方 (待 A 的 CAD)
- indoor_court.world / classroom_floor.world：地面、白線顏色照實拍；黃毛線外觀校正到「開始看到黃線的距離」跟實測一樣
- run_real_car.sh / compare_real_car.py / plot_real_car.py；sim_down.sh 也關 ros2 launch 跟 robot_state_publisher
- 修正 Jetson 節點時鐘死結 (程序卡頓後 /joint_states 排隊 + 緩衝區滿時丟掉的畫面不推進時鐘 -> 停約 10 s)
- 結果 (B 邏輯、10 顆球、900 s)：室內球場 run180/176/177 撿到 9/9/10 顆，教室 run178 9 顆，四組都沒越過黃線；
  BALL 間隔中位數 0.243~0.247 s (實測 0.233)、EDGE near_y 0.54~0.57 (實測 0.512)
- 實測資料：實體車子程式碼/jetson_data_20261012 (只放 CSV/程式/模型參數，影片沒放)

Co-Authored-By: Claude Opus 5.5 <noreply@anthropic.com>

File: src/tennis_bot/urdf/simple_bot.urdf (robot description, URDF)
Before this commit: robot tennis_bot, 11 links, 10 joints
Joints:
- joint camera_joint: origin xyz=0.135 0.1 0.13 rpy=0 0 1.6399 -> xyz=0.135 0.20 0.18 rpy=0 0.3718 1.6399
