Commit message: 新車 v2：鏡頭仰角建議、滾輪轉速上限 bug、海綿/撿球、新車整合錄影、P 控制對照
- 鏡頭仰角 (experiments/camera_tilt，實驗數據/camera_tilt_20261026)：建議約 15° (12~15° 可)
  邊界停車 (巡邏 120 rpm)：15° 以下 0/10 越線、21.3° 3/10；角落測試 12°/15° 2/18、21.3° 9/18；
  18° 以上車頭入鏡；15° 以下球在 D 估 >30 cm 就出畫面 (B 的盲衝不觸發)。
  剩下的角落越線是 B 轉 ~113° (WHEEL_TRACK 0.243) + D 閘門要 0.5 s SAFE 才重新放行，不是仰角能解
- 新環境變數：V2_CAM_PITCH_DEG (cad_v2_to_urdf)、TENNISBOT_PATROL_RPM (stm32_b_node，B 新版 120)、
  TENNISBOT_PICK_AT_MOUTH (real_car_node，球進撿球口就算撿到，跟滾輪拆開測)、GUI_CAM_POSE / GUI_TRACK_XYZ (錄影視角)
- 修正：Gazebo contact_max_correcting_vel 預設 100 會把滾輪卡在 100 rad/s (955 rpm)、左右變同方向轉
  -> pickup_test.world 改 1000，真實 1218 rpm 才跑得出來 (之前 W 70/90 的撿球掃描無效)
- 海綿 (experiments/sponge，實驗數據/sponge_20261026)：舊車模擬的滾輪位置是照 27 g 影片對的，球沒有被夾住，
  不能拿來校正；新車照 CAD 會夾 ~1 cm，真實轉速下 kp 2000/4000/8000 = 0/3、1/3、3/3 進車廂 (kp 待實測)
- 新車整合 + 錄影 (experiments/demo，影片不放 git，太大)：kp 8000 (暫定)、滾輪 1218 rpm、鏡頭 15°、巡邏 120 rpm、57.7 g
  B 點放：run201 3/10 出界、run202 7/10 出界、run198 7/10 出界；
  Sean 的連續 P 控制 (Kp 0.6)：run206 230 s 撿滿 10/10、沒出界 (每顆追球 ~16 s vs 點放 ~61 s，各 1 趟)
  路徑圖放在 影片/；中途作廢的 run199/200/203/205 沒放

Co-Authored-By: Claude Opus 5.5 <noreply@anthropic.com>

File: src/tennis_bot/urdf/tennis_bot_v2.urdf (robot description, URDF)
Before this commit: robot tennis_bot, 10 links, 9 joints
Joints:
- joint camera_joint: origin xyz=0.1030 0.0000 0.2222 rpy=0 0.3718 0.0691 -> xyz=0.1030 0.0000 0.2222 rpy=0 0.3717551306747922 0.0691
